File: REF1329_Altera.kicad_sch (KiCad schematic)
At the start: 38 parts, among them J1 DB25_Male, J3 Edge_Connector, J4 Edge_Connector, J6 Conn_02x05_Odd_Even, SW1 SW_Push, U1 SST28LF040, U2 SST28LF040, U3 HDSP-7501, U4 74HC164, U5 74HC04, U6 74HC374, U7 EPM240T100, X1 ASCO

Commit message: Add files via upload
Parts:
- removed X1: ASCO, N64_Hole:50 Mhz Crystal, symbol Oscillator:ASCO
Connections:
- net CLK: no longer names the net of U7.12 (IO1_12/GCLK0)
- no-connect marks 0 -> 1
