File: REF1329_Altera.kicad_pcb (KiCad board)
At the start: 2 copper layers, 102 x 71 mm, 42 parts, among them J1 DB25_Male, J3 Edge_Connector, J4 Edge_Connector, J6 Conn_02x05_Odd_Even, SW1 SW_Push, U1 SST28LF040, U2 SST28LF040, U3 HDSP-7501, U4 74HC164, U5 74HC04, U6 74HC374, U7 EPM240T100, X1 ASCO

Commit message: Add files via upload
Parts:
- removed X1: ASCO, N64_Hole:50 Mhz Crystal
Connections:
- U7 pad 12: /CLK -> unconnected-(U7-IO1_12/GCLK0-Pad12)
Routing:
- net /GND: track 535.7 -> 512.4 mm, vias 16 -> 15
- net /CLK: track 12.7 -> 0.00 mm, vias 2 -> 0
- net /VCC: track 446.2 -> 445.5 mm

Commit message: Add files via upload
Other:
- board text added: "1 cm Tall Push Button"
- board text added: "LibreShark Pro for N64 OSH REF1329 clone by github.com/RWeick 2026-10-25T12:07:00Z"
- board text removed: "1mm Tall Push Button"
- board text removed: "LibreShark Pro for N64 OSH REF1329 clone by github.com/RWeick 2023-05-17T16:40:00Z"
